File: Arduino_Mega2560_Practice/Section_01_USB_ATmega16U2.kicad_sch (KiCad schematic)
At the start: 0 parts

Commit message: USB部分
Parts:
- added C10: 1uF, Capacitor_SMD:C_0603_1608Metric, symbol Arduino_Mega2560_Lib:C_SMD_0603
- added C14, C15: 22P, Capacitor_SMD:C_0603_1608Metric, symbol Arduino_Mega2560_Lib:C_SMD_0603
- added C8: 100nf, Capacitor_SMD:C_0603_1608Metric, symbol Device:C
- added C9: 100nF, Capacitor_SMD:C_0603_1608Metric, symbol Arduino_Mega2560_Lib:C_SMD_0603
- added D2: D, Diode_SMD:D_1206_3216Metric, symbol Arduino_Mega2560_Lib:D_1206
- added F1: MF-MSMF050-2, Fuse:Fuse_1812_4532Metric_Pad1.30x3.40mm_HandSolder, symbol Device:Fuse
- added FB1: FerriteBead, Inductor_SMD:L_0805_2012Metric, symbol Arduino_Mega2560_Lib:FerriteBead_0805
- added J1: USB_C_Receptacle_USB2.0_16P, Connector_USB:USB_C_Receptacle_GCT_USB4105-xx-A_16P_TopMnt_Horizontal, symbol Arduino_Mega2560_Lib:USB_C_16P
- added J2: Conn_02x03_Odd_Even, Connector_PinHeader_2.54mm:PinHeader_2x03_P2.54mm_Vertical, symbol Arduino_Mega2560_Lib:Header_2x03
- added JP1: SolderJumper_2_Open, Jumper:SolderJumper-2_P1.3mm_Open_Pad1.0x1.5mm, symbol Arduino_Mega2560_Lib:SolderJumper_2
- added R2: 1M, Resistor_SMD:R_0603_1608Metric, symbol Arduino_Mega2560_Lib:R_SMD_0603
- added R3, R4: 5K1, Resistor_SMD:R_0603_1608Metric, symbol Device:R
- added RN2A, RN2D: 22R, Resistor_THT:R_Array_SIP8, symbol Device:R
- added RN5: 10K, Resistor_SMD:R_Array_Convex_4x0612, symbol Arduino_Mega2560_Lib:RArray_4x0612
- added RV1, RV2: Varistor, Resistor_SMD:R_0603_1608Metric, symbol Arduino_Mega2560_Lib:Varistor_0603
- added U1: ATMEGA16U2-MU, Package_DFN_QFN:VQFN-32-1EP_5x5mm_P0.5mm_EP3.1x3.1mm, symbol Arduino_Mega2560_Lib:ATmega16U2_MU
- added Y1: Crystal, Crystal:Crystal_HC49-4H_Vertical, symbol Arduino_Mega2560_Lib:Crystal_HC49
Connections:
- new net: C14.2, R2.2, U1.1 (XTAL1), Y1.1
- new net: C15.2, R2.1, U1.2 (PC0), Y1.2
- new net: FB1.2, J1.A1 (GND), J1.A12 (GND), J1.B1 (GND), J1.B12 (GND)
- new net: F1.2, J1.A4 (VBUS), J1.A9 (VBUS), J1.B4 (VBUS), J1.B9 (VBUS)
- new net +5V: C9.1, D2.1 (K), J2.2 (Pin_2), RN5.7 (R2.2), U1.32 (AVCC), U1.4 (VCC)
- new net CC1: J1.A5 (CC1), R3.1
- new net CC2: J1.B5 (CC2), R4.1
- new net D+: J1.A6 (D+), J1.B6 (D+), RN2D.1, RV2.1
- new net D-: J1.A7 (D-), J1.B7 (D-), RN2A.1, RV1.1
- new net GND: C14.1, C15.1, C8.1, C9.2, J2.6 (Pin_6), JP1.2 (B), R3.2, R4.2, U1.3 (GND), U1.33 (EXP)
- new net MISO2: J2.1 (Pin_1), U1.17 (PB3)
- new net MOSI2: J2.4 (Pin_4), U1.16 (PB2)
- new net RD+: RN2D.2, U1.29 (D+)
- new net RD-: RN2A.2, U1.30 (D-)
- new net RESET2: D2.2 (A), J2.5 (Pin_5), RN5.2 (R2.1), U1.24 (PC1//~{RESET})
- new net SCK2: J2.3 (Pin_3), U1.15 (PB1)
- new net UGND: C10.2, FB1.1, J1.S1 (SHIELD), JP1.1 (A), RV1.2, RV2.2, U1.28 (UGND)
- new net USBVCC: C8.2, F1.1, U1.31 (UVCC)
- new net VUCAP: C10.1, U1.27 (UCAP)
- no-connect marks 0 -> 2
