File: Arduino_Mega2560_Practice/Section_01_USB_ATmega16U2.kicad_sch (KiCad schematic)
At the start: 34 parts, among them J1 USB_C_Receptacle_USB2.0_16P, J2 Conn_02x03_Odd_Even, J3 Conn_02x02_Odd_Even, U1 ATMEGA16U2-MU, Y1 Crystal

Commit message: power
Parts:
- RN5: value 10K -> 10k
Changed lines of the file:
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@@
 			)
 		)
-		(property "Value" "10K"
+		(property "Value" "10k"
 			(at 146.05 82.296 90)
 			(show_name no)
